File: hardware/USBMux.kicad_sch (KiCad schematic)
At the start: 37 parts, among them J1 USB_0, J2 USB_1, J3 USB_A, J4 USB_C_Receptacle, SW1 SW_Push, SW2 SW_Push, U1 STM32F042F4Px, U10 USBLC6-2SC6, U2 FSUSB42MUX, U3 TPS2051CDBV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

Commit message: Update PCB, fix bug in BOOT0
Parts:
- added D1, D2, D3: LED, LED_SMD:LED_0805_2012Metric_Pad1.15x1.40mm_HandSolder, symbol Device:LED
- added H4: MountingHole_Pad, MountingHole:MountingHole_3.2mm_M3_DIN965_Pad, symbol Mechanical:MountingHole_Pad
- added R10, R11, R9: 150, Resistor_SMD:R_0805_2012Metric_Pad1.20x1.40mm_HandSolder, symbol Device:R
Connections:
- net BOOT0: now also U1.1 (PB8); no longer U1.14 (PB1)
- net GNDREF: now also H4.1
- net VCC: now also R10.1, R11.1, R9.1
- net HOST_1_ACTIVE: now reaches U1.12 (PA6)
- net HOST_1_ACTIVE: now also D1.1 (K)
- net HOST_2_ACTIVE: now reaches U1.13 (PA7)
- net HOST_2_ACTIVE: now also D2.1 (K)
- net DEVICE_POWERED: now reaches U1.19 (PA13)
- net DEVICE_POWERED: now also D3.1 (K)
- new net: D3.2 (A), R11.2
- new net: D1.2 (A), R9.2
- new net: D2.2 (A), R10.2
- no-connect marks 17 -> 14
Other:
- moved on the sheet: H1, H2, H3, J3, R6, SW2, U7
